File: pcb/VLF5.kicad_pcb (KiCad board)
At the start: 6 copper layers, 34 x 56 mm, 105 parts, among them CN1 532610571, J1 Conn_01x02_Pin, Q1 SS8050, Q3 SS8050, Q4 SS8050, Q5 SI7232DN-T1-GE3, U1 STM32H743VIHx, U10 LSM6DSMTR, U11 LIS2MDL, U12 BWU.FL-IPEX1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

Commit message: Playing with Trace Configurations
Still WIP!
Parts:
- moved RBOOT1 13.3 mm to (103.7, 63.8)
- moved C32 11.9 mm to (97.9, 61.4)
- moved C33 11.9 mm to (99.4, 62.4)
- moved C31 11.9 mm to (99.4, 64.3)
- moved C34 11.9 mm to (101.6, 61.8)
- moved C35 11.9 mm to (102.6, 63.8)
- moved C37 11.9 mm to (100.6, 62.7)
- moved C38 11.9 mm to (101.6, 63.7)
- moved C40 11.9 mm to (98.3, 62.8)
- moved C4 4.07 mm to (102.3, 77.3)
- moved C6 4.07 mm to (106.2, 77.0)
- moved C7 4.07 mm to (104.6, 77.0)
- moved C8 4.07 mm to (107.8, 77.0)
- moved L1 4.07 mm to (100.6, 79.2)
- moved L2 4.07 mm to (105.3, 74.0)
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Routing:
- net Net-(J_CAN1-Pin_2): track 0.00 -> 27.6 mm, vias 0 -> 1
- net Net-(J_CAN1-Pin_1): track 0.00 -> 26.9 mm, vias 0 -> 1
- net Net-(J_CAN1-Pin_3): track 0.00 -> 26.1 mm, vias 0 -> 1
- net Net-(J_CAN1-Pin_4): track 0.00 -> 25.5 mm, vias 0 -> 1
- net /SWDCLK: track 9.07 -> 20.8 mm
- net /CAN_TX: track 0.57 -> 11.5 mm
- net /GPS_nRST: track 10.9 -> 0.00 mm
- net /CAN_RX: track 0.57 -> 10.7 mm
- net /VBUS: track 0.57 -> 8.05 mm
- net /nRST: track 12.0 -> 18.2 mm, vias 0 -> 2
- net /LORA_MOSI: track 12.7 -> 18.8 mm
- net /Pyro/PYRO1: track 5.70 -> 0.00 mm
- net /MAG_SCL: track 1.91 -> 7.33 mm
- net /IMU_CLK: track 1.79 -> 6.76 mm
- net /BARO_CS: track 4.79 -> 0.00 mm
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