File: pcb/VLF5.kicad_pcb (KiCad board)
At the start: 6 copper layers, 34 x 56 mm, 105 parts, among them CN1 532610571, J1 Conn_01x02_Pin, Q1 SS8050, Q3 SS8050, Q4 SS8050, Q5 SI7232DN-T1-GE3, U1 STM32H743VIHx, U10 LSM6DSMTR, U11 LIS2MDL, U12 BWU.FL-IPEX1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

Commit message: VLF5 Rough Finish
Hallelujah
Connections:
- U1 pad G9: /PYRO_nEN -> unconnected-(U1-PD11-PadG9)
- U1 pad H9: /PYRO_PG -> unconnected-(U1-PD10-PadH9)
- U1 pad J2: unconnected-(U1-PA2-PadJ2) -> /LED_B_CTRL
- U1 pad J6: unconnected-(U1-PE12-PadJ6) -> /PYRO2_CONT
- U1 pad K10: /PYRO2_CONT -> unconnected-(U1-PD12-PadK10)
- U1 pad K2: /LED_B_CTRL -> /PS
- U1 pad K5: unconnected-(U1-PE9-PadK5) -> /PYRO_nEN
- U1 pad K6: /PS -> /PYRO_PG
Routing:
- net /LORA_TXEN: track 6.08 -> 31.3 mm, vias 1 -> 2
- net /LORA_RXEN: track 6.48 -> 31.3 mm, vias 1 -> 2
- net /LORA_BUSY: track 8.78 -> 33.4 mm, vias 2 -> 4
- net /LORA_CS: track 6.83 -> 28.5 mm, vias 1 -> 2
- net /SWDIO: track 7.21 -> 28.5 mm, vias 1 -> 2
- net /SWDCLK: track 6.98 -> 27.3 mm, vias 0 -> 2
- net /LORA_nRST: track 9.73 -> 24.7 mm
- net /LORA_SCK: track 11.9 -> 26.2 mm
- net /LORA_DIO1: track 9.25 -> 23.4 mm, vias 1 -> 3
- net /GPS_RX: track 5.22 -> 18.8 mm, vias 0 -> 3
- net /LORA_MISO: track 21.2 -> 33.0 mm, vias 2 -> 3
- net /GPS_TX: track 8.27 -> 19.7 mm, vias 0 -> 3
- net Net-(J_PYRO1-Pin_3): track 9.41 -> 17.9 mm
- net /LORA_MOSI: track 26.0 -> 32.9 mm
- net /GPS_nRST: track 10.5 -> 16.4 mm
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
Commit message: cleanup
Parts:
- added REF**: NetTie-2_SMD_Pad0.5mm, NetTie:NetTie-2_SMD_Pad0.5mm, B.Cu at (66.9, 61.1)
- moved C38 5.05 mm to (70.2, 64.9), turned to 0 degrees
- moved LED2 1.85 mm to (53.6, 83.1)
- moved R25 0.75 mm to (52.8, 80.6)
- moved R24 0.75 mm to (52.8, 78.5)
- moved C30 0.74 mm to (62.7, 63.9), turned to 0 degrees
- moved R26 0.70 mm to (52.8, 82.7)
- moved J1 0.66 mm to (58.8, 82.5)
- moved C44 0.61 mm to (64.9, 64.8), turned to 0 degrees
- moved J_PYRO1 0.53 mm to (75.7, 80.9)
- moved C39 0.43 mm to (64.9, 65.7), turned to 0 degrees
- moved J_CAN1 0.41 mm to (76.5, 82.8)
- moved J_CAN2 0.37 mm to (61.3, 82.8)
Connections:
- C29 pad 1: GND -> GND2
- C30 pad 2: GND -> GND2
- U1 pad C2: GND -> GND2
- U1 pad D10: /GPS_RX -> /GPS_TX
- U1 pad H10: /GPS_TX -> /GPS_RX
Routing:
- net Net-(J_PYRO1-Pin_3): track 17.9 -> 0.00 mm, vias 2 -> 8
- net GND2: track 0.00 -> 17.4 mm, vias 0 -> 19
- net +3.3V: track 40.5 -> 30.5 mm
- net +BATT: track 31.0 -> 22.1 mm
- net Net-(J_CAN1-Pin_4): track 33.3 -> 27.6 mm, vias 3 -> 1
- net Net-(J_CAN1-Pin_1): track 31.6 -> 26.4 mm, vias 2 -> 1
- net /Pyro/PYRO1: track 14.3 -> 9.39 mm
- net /nRST: track 22.3 -> 27.2 mm
- net +3.3VA: track 9.88 -> 5.09 mm
- net /Pyro/PYRO2: track 15.5 -> 11.7 mm
- net Net-(J_CAN1-Pin_3): track 28.6 -> 25.7 mm
- net Net-(J_CAN1-Pin_2): track 29.9 -> 27.2 mm, vias 3 -> 1
- net GND: track 4.79 -> 2.47 mm, vias 91 -> 163
- net /GPS_TX: track 19.7 -> 17.5 mm
- net /IMU_MOSI: track 10.9 -> 12.4 mm
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- added copper zone on F.Cu, net +BATT
- added copper zone on F.Cu, net /Pyro/PYRO1
- added copper zone on F.Cu, net /Pyro/PYRO2
- added copper zone on In1.Cu, net GND2
- added copper zone on B.Cu, net Net-(J_PYRO1-Pin_3)
- added copper zone on F.Cu, net Net-(J_PYRO1-Pin_3)
